Commit message: feat: Improve camera positioning for better workspace view
- Move camera to diagonal front-left position (0.8, 0.4, 0.3)
- Increase camera tilt from 28° to 40° for better downward view
- Adjust yaw to point towards table/workspace area
- Total camera height now ~0.83m for wider field of view

This should allow the camera to see both the robotic arm
and the table/objects in the workspace.

🤖 Generated with [Claude Code](https://claude.com/claude-code)

Co-Authored-By: Claude Opus 4.5 <noreply@anthropic.com>

File: ros_ws/src/kinova_llm_control/urdf/camera_stand.urdf.xacro (robot description, xacro)
@@ -67,6 +67,8 @@
                      color_fps="30"
                      visualize="false">
-    <!-- Camera tilted down to look at workspace -->
-    <origin xyz="0 0 0.02" rpy="0 0.5 3.14159"/>
+    <!-- Camera tilted down ~40 degrees to see workspace and table -->
+    <!-- rpy: roll=0, pitch=0.7rad (~40 deg down), yaw=2.8 (facing towards workspace center) -->
+    <!-- yaw slightly less than pi to point towards table area on the right -->
+    <origin xyz="0 0 0.02" rpy="0 0.7 2.8"/>
   </xacro:sensor_d435>
 </robot>

Commit message: fix: Center camera for full workspace visibility
Camera was positioned front-left but object was front-right.
New position:
- x=1.0m (further front for wider view)
- y=0.0m (centered to see both sides)
- z=0.5m (higher for bird's-eye perspective)
- pitch=45° down for workspace coverage
- yaw=π (facing back towards robot base)

Total camera height ~1.03m with stand, providing overhead
view of entire workspace including arm and surrounding objects.

🤖 Generated with [Claude Code](https://claude.com/claude-code)

Co-Authored-By: Claude Opus 4.5 <noreply@anthropic.com>

File: ros_ws/src/kinova_llm_control/urdf/camera_stand.urdf.xacro (robot description, xacro)
@@ -67,8 +67,8 @@
                      color_fps="30"
                      visualize="false">
-    <!-- Camera tilted down ~40 degrees to see workspace and table -->
-    <!-- rpy: roll=0, pitch=0.7rad (~40 deg down), yaw=2.8 (facing towards workspace center) -->
-    <!-- yaw slightly less than pi to point towards table area on the right -->
-    <origin xyz="0 0 0.02" rpy="0 0.7 2.8"/>
+    <!-- Camera tilted down ~45 degrees for overhead workspace view -->
+    <!-- rpy: roll=0, pitch=0.785rad (~45 deg down), yaw=pi (facing back towards robot) -->
+    <!-- Higher angle to see both arm and surrounding table/objects -->
+    <origin xyz="0 0 0.02" rpy="0 0.785 3.14159"/>
   </xacro:sensor_d435>
 </robot>

Commit message: feat: Add tabletop workspace with colored balls
New simulation environment:
- Table: 1.2m x 0.8m wooden table at 0.75m height
- Objects: 5 colored balls (red, green, blue, yellow, orange)
- Drop zone marker for placing objects
- Robot positioned at one end of table
- Camera at opposite end, looking across table

Layout mimics real-world tabletop pick-and-place setup:
- Robot can reach all balls
- Camera has full view of workspace
- Balls are colored for easy detection by vision system

Launch with: roslaunch kinova_llm_control tabletop_simulation.launch

🤖 Generated with [Claude Code](https://claude.com/claude-code)

Co-Authored-By: Claude Opus 4.5 <noreply@anthropic.com>

File: ros_ws/src/kinova_llm_control/urdf/camera_stand.urdf.xacro (robot description, xacro)
@@ -7,24 +7,24 @@
   <!-- Include the D435 camera macro -->
   <xacro:include filename="$(find realsense_gazebo_description)/urdf/_d435.urdf.xacro"/>
-  <!-- Camera stand base link -->
+  <!-- Camera stand base link - tripod style for tabletop mounting -->
   <link name="camera_stand_base">
     <visual>
       <geometry>
-        <cylinder radius="0.05" length="0.5"/>
+        <cylinder radius="0.04" length="0.35"/>
       </geometry>
-      <origin xyz="0 0 0.25" rpy="0 0 0"/>
-      <material name="grey">
-        <color rgba="0.5 0.5 0.5 1"/>
+      <origin xyz="0 0 0.175" rpy="0 0 0"/>
+      <material name="dark_metal">
+        <color rgba="0.2 0.2 0.2 1"/>
       </material>
     </visual>
     <collision>
       <geometry>
-        <cylinder radius="0.05" length="0.5"/>
+        <cylinder radius="0.04" length="0.35"/>
       </geometry>
-      <origin xyz="0 0 0.25" rpy="0 0 0"/>
+      <origin xyz="0 0 0.175" rpy="0 0 0"/>
     </collision>
     <inertial>
-      <mass value="1.0"/>
-      <inertia ixx="0.01" ixy="0" ixz="0" iyy="0.01" iyz="0" izz="0.01"/>
+      <mass value="0.5"/>
+      <inertia ixx="0.005" ixy="0" ixz="0" iyy="0.005" iyz="0" izz="0.005"/>
     </inertial>
   </link>
@@ -52,5 +52,5 @@
     <parent link="camera_stand_base"/>
     <child link="camera_mount"/>
-    <origin xyz="0 0 0.51" rpy="0 0 0"/>
+    <origin xyz="0 0 0.36" rpy="0 0 0"/>
   </joint>
   <!-- Attach D435 camera to mount -->
@@ -67,8 +67,8 @@
                      color_fps="30"
                      visualize="false">
-    <!-- Camera tilted down ~45 degrees for overhead workspace view -->
-    <!-- rpy: roll=0, pitch=0.785rad (~45 deg down), yaw=pi (facing back towards robot) -->
-    <!-- Higher angle to see both arm and surrounding table/objects -->
-    <origin xyz="0 0 0.02" rpy="0 0.785 3.14159"/>
+    <!-- Camera tilted slightly down to see table surface and objects -->
+    <!-- rpy: roll=0, pitch=0.3rad (~17 deg down), yaw=pi (facing back towards robot) -->
+    <!-- Positioned at table height, looking across at robot and objects -->
+    <origin xyz="0 0 0.02" rpy="0 0.3 3.14159"/>
   </xacro:sensor_d435>
 </robot>

Commit message: Add ball models and fix camera positioning for tabletop simulation
- Created SDF models for red, green, and blue balls (ball_red, ball_green, ball_blue)
- Added model.config files for Gazebo model recognition
- Added model.config for table model
- Shortened camera stand (0.35m -> 0.12m) for tabletop mounting
- Reduced camera tilt angle (0.3 -> 0.15 rad) for better table view
- Updated camera positions in both launch files
- Camera now sits on table surface looking back at robot and objects

🤖 Generated with [Claude Code](https://claude.com/claude-code)

Co-Authored-By: Claude Opus 4.5 <noreply@anthropic.com>

File: ros_ws/src/kinova_llm_control/urdf/camera_stand.urdf.xacro (robot description, xacro)
@@ -1,17 +1,17 @@
 <?xml version="1.0"?>
 <!--
-  Standalone RealSense D435 camera on a stand for Kinova simulation.
-  This creates a camera that can be spawned independently in Gazebo.
+  Standalone RealSense D435 camera on a short tabletop stand for Kinova simulation.
+  Designed to sit on the table surface and look across at the robot and objects.
 -->
 <robot name="camera_stand" xmlns:xacro="http://ros.org/wiki/xacro">
   <!-- Include the D435 camera macro -->
   <xacro:include filename="$(find realsense_gazebo_description)/urdf/_d435.urdf.xacro"/>
-  <!-- Camera stand base link - tripod style for tabletop mounting -->
+  <!-- Camera stand base - short tabletop tripod -->
   <link name="camera_stand_base">
     <visual>
       <geometry>
-        <cylinder radius="0.04" length="0.35"/>
+        <cylinder radius="0.03" length="0.12"/>
       </geometry>
-      <origin xyz="0 0 0.175" rpy="0 0 0"/>
+      <origin xyz="0 0 0.06" rpy="0 0 0"/>
       <material name="dark_metal">
         <color rgba="0.2 0.2 0.2 1"/>
@@ -20,11 +20,11 @@
     <collision>
       <geometry>
-        <cylinder radius="0.04" length="0.35"/>
+        <cylinder radius="0.03" length="0.12"/>
       </geometry>
-      <origin xyz="0 0 0.175" rpy="0 0 0"/>
+      <origin xyz="0 0 0.06" rpy="0 0 0"/>
     </collision>
     <inertial>
-      <mass value="0.5"/>
-      <inertia ixx="0.005" ixy="0" ixz="0" iyy="0.005" iyz="0" izz="0.005"/>
+      <mass value="0.3"/>
+      <inertia ixx="0.002" ixy="0" ixz="0" iyy="0.002" iyz="0" izz="0.002"/>
     </inertial>
   </link>
@@ -33,5 +33,5 @@
     <visual>
       <geometry>
-        <box size="0.1 0.1 0.02"/>
+        <box size="0.06 0.06 0.015"/>
       </geometry>
       <material name="dark_grey">
@@ -41,10 +41,10 @@
     <collision>
       <geometry>
-        <box size="0.1 0.1 0.02"/>
+        <box size="0.06 0.06 0.015"/>
       </geometry>
     </collision>
     <inertial>
-      <mass value="0.1"/>
-      <inertia ixx="0.001" ixy="0" ixz="0" iyy="0.001" iyz="0" izz="0.001"/>
+      <mass value="0.05"/>
+      <inertia ixx="0.0005" ixy="0" ixz="0" iyy="0.0005" iyz="0" izz="0.0005"/>
     </inertial>
   </link>
@@ -52,5 +52,5 @@
     <parent link="camera_stand_base"/>
     <child link="camera_mount"/>
-    <origin xyz="0 0 0.36" rpy="0 0 0"/>
+    <origin xyz="0 0 0.13" rpy="0 0 0"/>
   </joint>
   <!-- Attach D435 camera to mount -->
@@ -67,8 +67,7 @@
                      color_fps="30"
                      visualize="false">
-    <!-- Camera tilted slightly down to see table surface and objects -->
-    <!-- rpy: roll=0, pitch=0.3rad (~17 deg down), yaw=pi (facing back towards robot) -->
-    <!-- Positioned at table height, looking across at robot and objects -->
-    <origin xyz="0 0 0.02" rpy="0 0.3 3.14159"/>
+    <!-- Camera orientation: facing back towards robot (-x direction) with slight downward tilt -->
+    <!-- rpy: roll=0, pitch=0.15rad (~8.6 deg down), yaw=pi (facing back towards robot) -->
+    <origin xyz="0 0 0.02" rpy="0 0.15 3.14159"/>
   </xacro:sensor_d435>
 </robot>

Commit message: Fix robot position and camera height in simulation
- Robot: Spawn ON table edge (x=-0.05, z=0.75) instead of floor origin
- Camera stand: Increase height from 12cm to 50cm for better workspace view
- Camera tilt: Adjust from 8.6° to 26° down for proper coverage
- Direct robot spawn replaces kinova_gazebo include (enables position args)

🤖 Generated with [Claude Code](https://claude.com/claude-code)

Co-Authored-By: Claude Opus 4.5 <noreply@anthropic.com>

File: ros_ws/src/kinova_llm_control/urdf/camera_stand.urdf.xacro (robot description, xacro)
@@ -1,17 +1,19 @@
 <?xml version="1.0"?>
 <!--
-  Standalone RealSense D435 camera on a short tabletop stand for Kinova simulation.
-  Designed to sit on the table surface and look across at the robot and objects.
+  Standalone RealSense D435 camera on an elevated stand for Kinova simulation.
+  Designed to sit on the table surface with elevated view looking down at the entire workspace.
+  Stand height: 50cm (provides overhead view of table and robot)
+  Camera total height above table: ~52cm
 -->
 <robot name="camera_stand" xmlns:xacro="http://ros.org/wiki/xacro">
   <!-- Include the D435 camera macro -->
   <xacro:include filename="$(find realsense_gazebo_description)/urdf/_d435.urdf.xacro"/>
-  <!-- Camera stand base - short tabletop tripod -->
+  <!-- Camera stand base - tall tripod for elevated view -->
   <link name="camera_stand_base">
     <visual>
       <geometry>
-        <cylinder radius="0.03" length="0.12"/>
+        <cylinder radius="0.03" length="0.50"/>
       </geometry>
-      <origin xyz="0 0 0.06" rpy="0 0 0"/>
+      <origin xyz="0 0 0.25" rpy="0 0 0"/>
       <material name="dark_metal">
         <color rgba="0.2 0.2 0.2 1"/>
@@ -20,11 +22,11 @@
     <collision>
       <geometry>
-        <cylinder radius="0.03" length="0.12"/>
+        <cylinder radius="0.03" length="0.50"/>
       </geometry>
-      <origin xyz="0 0 0.06" rpy="0 0 0"/>
+      <origin xyz="0 0 0.25" rpy="0 0 0"/>
     </collision>
     <inertial>
-      <mass value="0.3"/>
-      <inertia ixx="0.002" ixy="0" ixz="0" iyy="0.002" iyz="0" izz="0.002"/>
+      <mass value="0.5"/>
+      <inertia ixx="0.01" ixy="0" ixz="0" iyy="0.01" iyz="0" izz="0.002"/>
     </inertial>
   </link>
@@ -52,5 +54,5 @@
     <parent link="camera_stand_base"/>
     <child link="camera_mount"/>
-    <origin xyz="0 0 0.13" rpy="0 0 0"/>
+    <origin xyz="0 0 0.51" rpy="0 0 0"/>
   </joint>
   <!-- Attach D435 camera to mount -->
@@ -67,7 +69,8 @@
                      color_fps="30"
                      visualize="false">
-    <!-- Camera orientation: facing back towards robot (-x direction) with slight downward tilt -->
-    <!-- rpy: roll=0, pitch=0.15rad (~8.6 deg down), yaw=pi (facing back towards robot) -->
-    <origin xyz="0 0 0.02" rpy="0 0.15 3.14159"/>
+    <!-- Camera orientation: facing back towards robot (-x direction) with moderate downward tilt -->
+    <!-- rpy: roll=0, pitch=0.45rad (~26 deg down), yaw=pi (facing back towards robot) -->
+    <!-- This angle provides good coverage of table surface and robot arm -->
+    <origin xyz="0 0 0.02" rpy="0 0.45 3.14159"/>
   </xacro:sensor_d435>
 </robot>

Commit message: Fix camera stand stability - make it static
- Add world link and fixed joint to prevent stand from falling over
- Camera stand is now fixed in place during simulation

🤖 Generated with [Claude Code](https://claude.com/claude-code)

Co-Authored-By: Claude Opus 4.5 <noreply@anthropic.com>

File: ros_ws/src/kinova_llm_control/urdf/camera_stand.urdf.xacro (robot description, xacro)
@@ -5,8 +5,11 @@
   Stand height: 50cm (provides overhead view of table and robot)
   Camera total height above table: ~52cm
+  NOTE: Stand is STATIC (fixed in place, does not fall over)
 -->
 <robot name="camera_stand" xmlns:xacro="http://ros.org/wiki/xacro">
   <!-- Include the D435 camera macro -->
   <xacro:include filename="$(find realsense_gazebo_description)/urdf/_d435.urdf.xacro"/>
+  <!-- World link for fixed base -->
+  <link name="world"/>
   <!-- Camera stand base - tall tripod for elevated view -->
   <link name="camera_stand_base">
@@ -31,4 +34,10 @@
     </inertial>
   </link>
+  <!-- Fix stand to world so it doesn't fall over -->
+  <joint name="world_to_stand" type="fixed">
+    <parent link="world"/>
+    <child link="camera_stand_base"/>
+    <origin xyz="0 0 0" rpy="0 0 0"/>
+  </joint>
   <!-- Camera mount on top of stand -->
   <link name="camera_mount">
